File: schematics/MC14490P_module/MC14490P_module.sch (KiCad schematic (older format))
At the start: 2 parts

Commit message: new
Parts:
- added J?: Conn_01x08_Female, symbol Connector:Conn_01x08_Female
Connections:
- net at U?.1 (AIN): now also J?.1 (Pin_1)
- net at U?.10 (FIN): now also J?.6 (Pin_6)
- net at U?.12 (DIN): now also J?.4 (Pin_4)
- net at U?.14 (BIN): now also J?.2 (Pin_2)
- net at U?.3 (CIN): now also J?.3 (Pin_3)
- net at U?.5 (EIN): now also J?.5 (Pin_5)
- net at U?.7 (OSCIN): now also J?.7 (Pin_7)
Changed lines of the file:
@@
 	-1   0    0    -1
 $EndComp
+$Comp
+L Connector:Conn_01x08_Female J?
+U 1 1 5ECD2EFF
+P 7710 2820
+F 0 "J?" H 7602 3305 50  0000 C CNN
+F 1 "Conn_01x08_Female" H 7602 3214 50  0000 C CNN
+F 2 "" H 7710 2820 50  0001 C CNN
+F 3 "~" H 7710 2820 50  0001 C CNN
+	1    7710 2820
+	1    0    0    -1
+$EndComp
+Wire Wire Line
+	3620 2550 5300 2550
+Wire Wire Line
+	3620 2650 5300 2650
+Wire Wire Line
+	3620 2750 5300 2750
+Wire Wire Line
+	5300 2850 3620 2850
+Wire Wire Line
+	3620 2950 5300 2950
+Wire Wire Line
+	5300 3050 3620 3050
+Wire Wire Line
+	3620 3150 5300 3150
 $EndSCHEMATC
